Commit message: fix gazebo 7.0 NaN bug on zero collision geometry

File: kinova_description/urdf/kinova_common.xacro (robot description, xacro)
@@ -46,10 +46,10 @@
             <visual>
                 <geometry>
-                    <box size = "0 0 0"/>
+                    <box size = "0.001 0.001 0.001"/>
                 </geometry>
             </visual>
             <collision>
                 <geometry>
-                    <box size = "0 0 0"/>
+                    <box size = "0.001 0.001 0.001"/>
                 </geometry>
             </collision>
